File: kicad/solderbit-segment-shift-edition.kicad_pcb (KiCad board)
At the start: 2 copper layers, 28 x 54 mm, 16 parts, among them J1 Conn_01x08_Pin, U1 74HC595D, U2 74HC595N

Commit message: Update all documentation
Parts:
- U2: value 74HC595N -> SN74HC595N
- moved DS1 9.16 mm to (140.0, 98.0)
Connections:
- net /RCLK renamed /STCP
- net /SER renamed /DS
- net /SRCLK renamed /SHCP
- net /~{SRCLR} renamed /~{MR}
Routing:
- net GND: vias 30 -> 32
