File: kicad/solderbit-segment-shift-edition.kicad_sch (KiCad schematic)
At the start: 15 parts, among them J1 Conn_01x08_Pin, U1 74HC595D, U2 74HC595N

Commit message: Update all documentation
Parts:
- removed U1: 74HC595D, Solderbit_Segment:SOIC-16_3.9x9.9mm_P1.27mm, symbol 74xx:74HC595
- added U1: 74HC595D, Solderbit_Segment:SOIC-16_3.9x9.9mm_P1.27mm, symbol Solderbit_Segment:74HC595_Nexperia
- DS1: Onecall (none) -> 3648330
- J1: LCSC Part (none) -> C492407; LCSC datasheet (none) -> https://www.lcsc.com/datasheet/C492407.pdf; Onecall 3049532 -> 1593416
- R1, R2: Onecall (none) -> 9241060
- U2: value 74HC595N -> SN74HC595N; LCSC datasheet (none) -> https://www.lcsc.com/datasheet/C507175.pdf
Connections:
- net A: now also U1.15 (Q0)
- net B: now also U1.1 (Q1)
- net C: now also U1.2 (Q2)
- net D: now also U1.3 (Q3)
- net E: now also U1.4 (Q4)
- net F: now also U1.5 (Q5)
- net G: now also U1.6 (Q6)
- net GND: now also U1.8 (GND)
- net H: now also U1.7 (Q7)
- net H': now also U1.9 (Q7S)
- net VCC: now also U1.16 (VCC)
- net ~{OE}: now also U1.13 (~{OE})
- net RCLK renamed STCP
- net STCP: now also U1.12 (STCP)
- net SER renamed DS
- net DS: now also U1.14 (DS)
- net SRCLK renamed SHCP
- net SHCP: now also U1.11 (SHCP)
- net ~{SRCLR} renamed ~{MR}
- net ~{MR}: now also U1.10 (~{MR})
Other:
- moved on the sheet: C1, R1, R2, U2

Commit message: Remove DNP flag for header pins
Parts:
- J1: now fitted
Changed lines of the file:
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@@
 	(text_box "You can choose between U1 (SOP-16) or U2 (DIP-16). Both are the same shift register in different packages. The larger through-hole DIP-16 is easier to solder for beginners, while the smaller SOP-16 offers a challenge for those with more experience."
 		(exclude_from_sim no)
-		(at 41.275 104.14 0)
+		(at 43.18 106.045 0)
 		(size 57.15 12.065)
 		(margins 0.9525 0.9525 0.9525 0.9525)
@@
 		(on_board yes)
 		(in_pos_files yes)
-		(dnp yes)
+		(dnp no)
 		(property "Reference" "J1"
 			(at 171.196 105.41 0)
